Commit message: FEB 17

File: install/ur_description/share/ur_description/urdf/inc/mop_tool.xacro (robot description, xacro)
@@ -7,24 +7,17 @@
       <origin xyz="-0.0 0.0 0.47" rpy="${pi/2} ${-pi} 0" />
     </joint>
-    <link name="${prefix}mop_handle">
-      <visual>
-        <origin xyz="0 0 0" rpy="0 0 0" />
-        <geometry>
-          <mesh filename="package://ur_description/meshes/mop_handle.obj" scale="0.0022 0.001 0.002" />
-        </geometry>
-        <material name="mop_purple"><color rgba="0.18 0.05 0.35 1" /></material>
-      </visual>
-      <collision>
-        <origin xyz="0 0.235 0" rpy="${pi/2} ${-pi} 0" />
-        <geometry>
-          <cylinder radius="0.015" length="0.47" />
-        </geometry>
-      </collision>
-      <inertial>
-        <mass value="0.5" />
-        <origin xyz="0 0 0" rpy="0 0 0" />
-        <inertia ixx="0.01" ixy="0" ixz="0" iyy="0.01" iyz="0" izz="0.01" />
-      </inertial>
-    </link>
+<link name="mop_handle">
+    <visual>
+      <origin rpy="0 0 0" xyz="0 -0.03 0"/>
+      <geometry>
+        <mesh filename="package://ur_description/meshes/mop_handle.obj" scale="0.0022 0.001 0.002"/>
+      </geometry>
+    </visual>
+    <inertial>
+      <mass value="0.5"/>
+      <origin rpy="0 0 0" xyz="0 0 0"/>
+      <inertia ixx="0.01" ixy="0" ixz="0" iyy="0.01" iyz="0" izz="0.01"/>
+    </inertial>
+  </link>
     <joint name="${prefix}mop_socket_roll" type="continuous">
       <parent link="${prefix}mop_handle" />

File: install/ur_description/share/ur_description/urdf/ur_for_ik.urdf (robot description, URDF)
Before this commit: robot ur_table_assembly, 29 links, 28 joints
Links:
- removed link ur_2_base
- removed link ur_2_base_link
- removed link ur_2_base_link_inertia
- removed link ur_2_flange
- removed link ur_2_forearm_link
- removed link ur_2_ft_frame
- removed link ur_2_shoulder_link
- removed link ur_2_tool0
- removed link ur_2_upper_arm_link
- removed link ur_2_wrist_1_link
- removed link ur_2_wrist_2_link
- removed link ur_2_wrist_3_link
- link mop_handle: geometry visual mesh filename=package://ur_description/meshes/mop_handle.obj scale=0.0022 0.001 0.002
- link table_link: geometry collision box size=1.32 0.72 0.60; visual mesh filename=package://ur_description/meshes/test.stl scale=1 1 1
Joints:
- removed joint ur_2_base_joint
- removed joint ur_2_base_link-base_fixed_joint
- removed joint ur_2_base_link-base_link_inertia
- removed joint ur_2_elbow_joint
- removed joint ur_2_flange-tool0
- removed joint ur_2_shoulder_lift_joint
- removed joint ur_2_shoulder_pan_joint
- removed joint ur_2_wrist_1_joint
- removed joint ur_2_wrist_2_joint
- removed joint ur_2_wrist_3-flange
- removed joint ur_2_wrist_3_joint
- removed joint ur_2_wrist_3_link-ft_frame
- joint base_joint: origin xyz=0 0 0.65 rpy=0 0 0 -> xyz=0 -0.1 0.65 rpy=0 0 0
- joint world_to_table: origin xyz=0.0 0.45 0.31 rpy=0 0 0 -> xyz=0.0 0.35 0.31 rpy=0 0 0

File: install/ur_description/share/ur_description/urdf/ur_mop_standalone.urdf.xacro (robot description, xacro)
@@ -1,4 +1,4 @@
 <?xml version="1.0"?>
-<robot xmlns:xacro="http://wiki.ros.org/xacro" name="ur_mop_standalone">
+<robot xmlns:xacro="http://wiki.ros.org/xacro" name="ur">
   <xacro:include filename="$(find ur_description)/urdf/ur_macro.xacro"/>
   <xacro:include filename="$(find ur_description)/urdf/inc/mop_tool.xacro"/>
@@ -25,6 +25,81 @@
     safety_k_position="$(arg safety_k_position)"
     >
-    <origin xyz="0 -0.2 0.81" rpy="0 0 0" />
+    <origin xyz="0 -0.1 0.65" rpy="0 0 0" />
   </xacro:ur_robot>
   <xacro:mop_tool prefix="" parent="tool0" />
+  <ros2_control name="GazeboSimSystem" type="system">
+    <hardware>
+      <plugin>gz_ros2_control/GazeboSimSystem</plugin>
+    </hardware>
+    <joint name="shoulder_pan_joint">
+      <command_interface name="position"/>
+      <state_interface name="position"/>
+      <state_interface name="velocity"/>
+    </joint>
+    <joint name="shoulder_lift_joint">
+      <command_interface name="position"/>
+      <state_interface name="position"/>
+      <state_interface name="velocity"/>
+    </joint>
+    <joint name="elbow_joint">
+      <command_interface name="position"/>
+      <state_interface name="position"/>
+      <state_interface name="velocity"/>
+    </joint>
+    <joint name="wrist_1_joint">
+      <command_interface name="position"/>
+      <state_interface name="position"/>
+      <state_interface name="velocity"/>
+    </joint>
+    <joint name="wrist_2_joint">
+      <command_interface name="position"/>
+      <state_interface name="position"/>
+      <state_interface name="velocity"/>
+    </joint>
+    <joint name="wrist_3_joint">
+      <command_interface name="position"/>
+      <state_interface name="position"/>
+      <state_interface name="velocity"/>
+    </joint>
+    <joint name="mop_socket_roll">
+      <state_interface name="position"/>
+      <state_interface name="velocity"/>
+    </joint>
+    <joint name="mop_socket_yaw">
+      <state_interface name="position"/>
+      <state_interface name="velocity"/>
+    </joint>
+  </ros2_control>
+<link name="table_link">
+    <visual>
+      <origin rpy="0 0 0" xyz="0.7 0.36 -0.3"/>
+      <geometry>
+        <mesh filename="package://ur_description/meshes/test.stl" scale="1 1 1"/>
+      </geometry>
+      <material name="table_material">
+        <color rgba="0.6 0.4 0.2 1"/>
+      </material>
+    </visual>
+    <collision>
+      <origin rpy="0 0 0" xyz="0.05 0 0.0"/>
+      <geometry>
+        <box size="1.32 0.72 0.60"/>
+      </geometry>
+    </collision>
+    <inertial>
+      <mass value="50"/>
+      <origin rpy="0 0 0" xyz="0.7 0.36 -0.3"/>
+      <inertia ixx="10" ixy="0" ixz="0" iyy="10" iyz="0" izz="5"/>
+    </inertial>
+  </link>
+  <joint name="world_to_table" type="fixed">
+    <parent link="world"/>
+    <child link="table_link"/>
+    <origin rpy="0 0 0" xyz="0.0 0.35 0.31"/>
+  </joint>
+  <gazebo>
+    <plugin filename="gz_ros2_control-system" name="gz_ros2_control::GazeboSimROS2ControlPlugin">
+      <parameters>$(find ur_description)/config/ur_controllers.yaml</parameters>
+    </plugin>
+  </gazebo>
 </robot>

Commit message: FEB 18 home

File: install/ur_description/share/ur_description/urdf/inc/mop_tool.xacro (robot description, xacro)
@@ -7,17 +7,24 @@
       <origin xyz="-0.0 0.0 0.47" rpy="${pi/2} ${-pi} 0" />
     </joint>
-<link name="mop_handle">
-    <visual>
-      <origin rpy="0 0 0" xyz="0 -0.03 0"/>
-      <geometry>
-        <mesh filename="package://ur_description/meshes/mop_handle.obj" scale="0.0022 0.001 0.002"/>
-      </geometry>
-    </visual>
-    <inertial>
-      <mass value="0.5"/>
-      <origin rpy="0 0 0" xyz="0 0 0"/>
-      <inertia ixx="0.01" ixy="0" ixz="0" iyy="0.01" iyz="0" izz="0.01"/>
-    </inertial>
-  </link>
+    <link name="${prefix}mop_handle">
+      <visual>
+        <origin xyz="0 0 0" rpy="0 0 0" />
+        <geometry>
+          <mesh filename="package://ur_description/meshes/mop_handle.obj" scale="0.0022 0.001 0.002" />
+        </geometry>
+        <material name="mop_purple"><color rgba="0.18 0.05 0.35 1" /></material>
+      </visual>
+      <collision>
+        <origin xyz="0 0.235 0" rpy="${pi/2} ${-pi} 0" />
+        <geometry>
+          <cylinder radius="0.015" length="0.47" />
+        </geometry>
+      </collision>
+      <inertial>
+        <mass value="0.5" />
+        <origin xyz="0 0 0" rpy="0 0 0" />
+        <inertia ixx="0.01" ixy="0" ixz="0" iyy="0.01" iyz="0" izz="0.01" />
+      </inertial>
+    </link>
     <joint name="${prefix}mop_socket_roll" type="continuous">
       <parent link="${prefix}mop_handle" />

File: install/ur_description/share/ur_description/urdf/ur_for_ik.urdf (robot description, URDF)
Before this commit: robot ur, 17 links, 16 joints
Links:
- added link ur_2_base
- added link ur_2_base_link
- added link ur_2_base_link_inertia, mass 4.0; collision mesh filename=package://ur_description/meshes/ur5e/collision/base.stl; visual mesh filename=package://ur_description/meshes/ur5e/visual/base.dae
- added link ur_2_flange
- added link ur_2_forearm_link, mass 2.846; collision mesh filename=package://ur_description/meshes/ur5e/collision/forearm.stl; visual mesh filename=package://ur_description/meshes/ur5e/visual/forearm.dae
- added link ur_2_ft_frame
- added link ur_2_shoulder_link, mass 3.761; collision mesh filename=package://ur_description/meshes/ur5e/collision/shoulder.stl; visual mesh filename=package://ur_description/meshes/ur5e/visual/shoulder.dae
- added link ur_2_tool0
- added link ur_2_upper_arm_link, mass 8.058; collision mesh filename=package://ur_description/meshes/ur5e/collision/upperarm.stl; visual mesh filename=package://ur_description/meshes/ur5e/visual/upperarm.dae
- added link ur_2_wrist_1_link, mass 1.37; collision mesh filename=package://ur_description/meshes/ur5e/collision/wrist1.stl; visual mesh filename=package://ur_description/meshes/ur5e/visual/wrist1.dae
- added link ur_2_wrist_2_link, mass 1.3; collision mesh filename=package://ur_description/meshes/ur5e/collision/wrist2.stl; visual mesh filename=package://ur_description/meshes/ur5e/visual/wrist2.dae
- added link ur_2_wrist_3_link, mass 0.365; collision mesh filename=package://ur_description/meshes/ur5e/collision/wrist3.stl; visual mesh filename=package://ur_description/meshes/ur5e/visual/wrist3.dae
- link mop_handle: geometry collision cylinder length=0.8 radius=0.015; visual mesh filename=package://ur_description/meshes/mop_handle.obj scale=0.002 0.0015 0.002
- link mop_head: geometry collision box size=0.35 0.2 0.04; visual mesh filename=package://ur_description/meshes/mop_base.obj scale=0.003 0.002 0.002
- link table_link: geometry collision box size=1.38 0.72 0.60; visual mesh filename=package://ur_description/meshes/test.stl scale=1 1 1
Joints:
- added joint ur_2_base_joint: type fixed, parent world, child ur_2_base_link, origin xyz=0.0 1.1 1.0 rpy=0 0 3.141592653589793
- added joint ur_2_base_link-base_fixed_joint: type fixed, parent ur_2_base_link, child ur_2_base, origin xyz=0 0 0 rpy=0 0 3.141592653589793
- added joint ur_2_base_link-base_link_inertia: type fixed, parent ur_2_base_link, child ur_2_base_link_inertia, origin xyz=0 0 0 rpy=0 0 3.141592653589793
- added joint ur_2_elbow_joint: type revolute, parent ur_2_upper_arm_link, child ur_2_forearm_link, origin xyz=-0.425 0 0 rpy=0 0 0, axis 0 0 1, limit lower=-3.141592653589793 upper=3.141592653589793 effort=150.0 velocity=3.141592653589793
- added joint ur_2_flange-tool0: type fixed, parent ur_2_flange, child ur_2_tool0, origin xyz=0 0 0 rpy=1.5707963267948966 0 1.5707963267948966
- added joint ur_2_shoulder_lift_joint: type revolute, parent ur_2_shoulder_link, child ur_2_upper_arm_link, origin xyz=0 0 0 rpy=1.570796327 0 0, axis 0 0 1, limit lower=-6.283185307179586 upper=6.283185307179586 effort=150.0 velocity=3.141592653589793
- added joint ur_2_shoulder_pan_joint: type revolute, parent ur_2_base_link_inertia, child ur_2_shoulder_link, origin xyz=0 0 0.1625 rpy=0 0 0, axis 0 0 1, limit lower=-6.283185307179586 upper=6.283185307179586 effort=150.0 velocity=3.141592653589793
- added joint ur_2_wrist_1_joint: type revolute, parent ur_2_forearm_link, child ur_2_wrist_1_link, origin xyz=-0.3922 0 0.1333 rpy=0 0 0, axis 0 0 1, limit lower=-6.283185307179586 upper=6.283185307179586 effort=28.0 velocity=3.141592653589793
- added joint ur_2_wrist_2_joint: type revolute, parent ur_2_wrist_1_link, child ur_2_wrist_2_link, origin xyz=0 -0.0997 -2.044881182297852e-11 rpy=1.570796327 0 0, axis 0 0 1, limit lower=-6.283185307179586 upper=6.283185307179586 effort=28.0 velocity=3.141592653589793
- added joint ur_2_wrist_3-flange: type fixed, parent ur_2_wrist_3_link, child ur_2_flange, origin xyz=0 0 0 rpy=0 -1.5707963267948966 -1.5707963267948966
- added joint ur_2_wrist_3_joint: type revolute, parent ur_2_wrist_2_link, child ur_2_wrist_3_link, origin xyz=0 0.0996 -2.042830148012698e-11 rpy=1.570796326589793 3.141592653589793 3.141592653589793, axis 0 0 1, limit lower=-6.283185307179586 upper=6.283185307179586 effort=28.0 velocity=3.141592653589793
- added joint ur_2_wrist_3_link-ft_frame: type fixed, parent ur_2_wrist_3_link, child ur_2_ft_frame, origin xyz=0 0 0 rpy=3.141592653589793 0 0
- joint base_joint: origin xyz=0 -0.1 0.65 rpy=0 0 0 -> xyz=0 0 0.65 rpy=0 0 0
- joint mop_mount_joint: origin xyz=-0.0 0.0 0.47 rpy=1.5707963267948966 -3.141592653589793 0 -> xyz=-0.0 0.0 0.6 rpy=1.5707963267948966 -3.141592653589793 0
- joint world_to_table: origin xyz=0.0 0.35 0.31 rpy=0 0 0 -> xyz=0.0 0.45 0.31 rpy=0 0 0

File: install/ur_description/share/ur_description/urdf/ur_macro.xacro (robot description, xacro)
@@ -74,5 +74,5 @@
     <link name="${tf_prefix}base_link_inertia">
       <visual>
-        <origin xyz="0 0 0" rpy="0 0 ${pi}"/>
+        <origin xyz="0 0 0" rpy="0 0 0"/>
         <geometry>
           <xacro:get_mesh name="base" type="visual"/>
@@ -80,5 +80,5 @@
       </visual>
       <collision>
-        <origin xyz="0 0 0" rpy="0 0 ${pi}"/>
+        <origin xyz="0 0 0" rpy="0 0 0"/>
         <geometry>
           <xacro:get_mesh name="base" type="collision"/>

File: install/ur_description/share/ur_description/urdf/ur_mop_standalone.urdf.xacro (robot description, xacro)
@@ -28,4 +28,18 @@
   </xacro:ur_robot>
   <xacro:mop_tool prefix="" parent="tool0" />
+    <xacro:ur_robot
+    name="ur_2"
+    tf_prefix="ur_2_"
+    parent="world"
+    joint_limits_parameters_file="$(arg joint_limit_params)"
+    kinematics_parameters_file="$(arg kinematics_params)"
+    physical_parameters_file="$(arg physical_params)"
+    visual_parameters_file="$(arg visual_params)"
+    safety_limits="$(arg safety_limits)"
+    safety_pos_margin="$(arg safety_pos_margin)"
+    safety_k_position="$(arg safety_k_position)"
+    >
+    <origin xyz="0.0 1.1 1.0" rpy="0 0 ${pi}" />
+  </xacro:ur_robot>
   <ros2_control name="GazeboSimSystem" type="system">
     <hardware>
@@ -70,4 +84,10 @@
       <state_interface name="velocity"/>
     </joint>
+    <joint name="ur_2_shoulder_pan_joint"><command_interface name="position"/><state_interface name="position"/><state_interface name="velocity"/></joint>
+    <joint name="ur_2_shoulder_lift_joint"><command_interface name="position"/><state_interface name="position"/><state_interface name="velocity"/></joint>
+    <joint name="ur_2_elbow_joint"><command_interface name="position"/><state_interface name="position"/><state_interface name="velocity"/></joint>
+    <joint name="ur_2_wrist_1_joint"><command_interface name="position"/><state_interface name="position"/><state_interface name="velocity"/></joint>
+    <joint name="ur_2_wrist_2_joint"><command_interface name="position"/><state_interface name="position"/><state_interface name="velocity"/></joint>
+    <joint name="ur_2_wrist_3_joint"><command_interface name="position"/><state_interface name="position"/><state_interface name="velocity"/></joint>
   </ros2_control>
 <link name="table_link">
