Commit message: working robot 1 but not robot 2

File: src/robotiq_description/urdf/2f_140.ros2_control.xacro (robot description, xacro)
@@ -10,5 +10,5 @@
         use_fake_hardware:=false
         mock_sensor_commands:=false
-        com_port:=/dev/ttyUSB0
+        com_port:=/tmp/ttyUR
         gripper_speed_multiplier:=1.0
         gripper_force_multiplier:=0.5

File: src/robotiq_description/urdf/robotiq_2f_140_gripper.urdf.xacro (robot description, xacro)
@@ -3,5 +3,5 @@
     <!-- parameters -->
     <xacro:arg name="use_fake_hardware" default="true" />
-    <xacro:arg name="com_port" default="/dev/ttyUSB0" />
+    <xacro:arg name="com_port" default="/tmp/ttyUR" />
     <!-- Import macros -->
     <xacro:include filename="$(find robotiq_description)/urdf/robotiq_2f_140_macro.urdf.xacro" />

File: src/robotiq_description/urdf/robotiq_2f_140_macro.urdf.xacro (robot description, xacro)
@@ -13,5 +13,5 @@
         mock_sensor_commands:=false
         include_ros2_control:=true
-        com_port:=/dev/ttyUSB0
+        com_port:=//tmp/ttyUR
         gripper_speed_multiplier:=1.0
         gripper_force_multiplier:=0.5

File: src/robotiq_description/urdf/robotiq_2f_85_macro.urdf.xacro (robot description, xacro)
@@ -13,5 +13,5 @@
         mock_sensor_commands:=false
         include_ros2_control:=true
-        com_port:=/dev/ttyUSB0
+        com_port:=/tmp/ttyUR
         gripper_speed_multiplier:=1.0
         gripper_force_multiplier:=0.5

File: src/ur_description/urdf/inc/mop_tool.xacro (robot description, xacro)
@@ -5,18 +5,18 @@
       <parent link="${parent}" />
       <child link="${prefix}mop_handle" />
-      <origin xyz="-0.0 0.0 0.47" rpy="${pi/2} ${-pi} 0" />
+      <origin xyz="-0.0 0.0 0.245" rpy="${pi/2} ${-pi} 0" />
     </joint>
     <link name="${prefix}mop_handle">
       <visual>
-        <origin xyz="0 0.1 0" rpy="0 0 0" />
+        <origin xyz="0 0 0" rpy="${pi/2} ${-pi} 0" />
         <geometry>
-          <mesh filename="package://ur_description/meshes/mop_handle.obj" scale="0.0022 0.00095 0.002" />
+          <cylinder radius="0.015" length="0.49" />
         </geometry>
-        <material name="mop_purple"><color rgba="0.18 0.05 0.35 1" /></material>
+        <material name="mop_purple"><color rgba="0.7 0.7 0.7 1" /></material>
       </visual>
       <collision>
-        <origin xyz="0 0.35 0" rpy="${pi/2} ${-pi} 0" />
+        <origin xyz="0 0 0" rpy="${pi/2} ${-pi} 0" />
         <geometry>
-          <cylinder radius="0.015" length="0.25" />
+          <cylinder radius="0.015" length="0.49" />
         </geometry>
       </collision>
@@ -31,5 +31,5 @@
       <child link="${prefix}mop_dummy_r" />
       <axis xyz="1 0 0" />
-      <origin xyz="0 -0.0 -0.0" rpy="0 0 0" />
+      <origin xyz="0 -0.245 -0.0" rpy="0 0 0" />
       <dynamics damping="0.5" friction="0.01"/>
     </joint>
@@ -48,5 +48,5 @@
     <link name="${prefix}mop_head">
       <visual>
-        <origin xyz="0 0.2 -0.07" rpy="0 0 0" />
+        <origin xyz="-0.01 -0.01 -0.07" rpy="0 0 0" />
         <geometry>
           <mesh filename="package://ur_description/meshes/mop_base.obj" scale="0.002 0.001 0.0015" />
@@ -55,5 +55,5 @@
       </visual>
       <collision>
-        <origin xyz="0 0.2 -0.0" rpy="${pi/2} ${-pi} 0"  />
+        <origin xyz="0 0 -0.0" rpy="${pi/2} ${-pi} 0"  />
         <geometry>
           <box size="0.25 0.13 0.02" />

File: src/ur_description/urdf/ur_mop_standalone.urdf.xacro (robot description, xacro)
@@ -8,8 +8,10 @@
   <xacro:arg name="ur_type" default="ur5"/>
   <xacro:arg name="tf_prefix" default="" />
+  <xacro:arg name="tf_prefix_2" default="ur_2_" />
   <xacro:arg name="name" default="ur"/>
   <xacro:arg name="use_gazebo" default="false"/>
   <xacro:arg name="joint_limit_params" default="$(find ur_description)/config/$(arg ur_type)/joint_limits.yaml"/>
   <xacro:arg name="kinematics_params" default="$(find ur_description)/config/$(arg ur_type)/default_kinematics.yaml"/>
+  <xacro:arg name="kinematics_params_2" default="$(find ur_description)/config/$(arg ur_type)/default_kinematics_2.yaml"/>
   <xacro:arg name="physical_params" default="$(find ur_description)/config/$(arg ur_type)/physical_parameters.yaml"/>
   <xacro:arg name="visual_params" default="$(find ur_description)/config/$(arg ur_type)/visual_parameters.yaml"/>
@@ -17,5 +19,6 @@
   <xacro:arg name="safety_pos_margin" default="0.15"/>
   <xacro:arg name="safety_k_position" default="20"/>
-  <xacro:arg name="robot_ip" default="192.168.1.103"/>
+  <xacro:arg name="robot_ip" default="192.168.1.104"/>
+  <xacro:arg name="robot_2_ip" default="192.168.1.103"/>
   <xacro:arg name="use_mock_hardware" default="false"/>
   <xacro:arg name="mock_sensor_commands" default="false"/>
@@ -29,5 +32,9 @@
   <xacro:arg name="script_sender_port" default="50002"/>
   <xacro:arg name="trajectory_port" default="50003"/>
-  <xacro:arg name="use_tool_communication" default="false"/>
+  <xacro:arg name="script_command_port_2" default="50014"/>
+  <xacro:arg name="reverse_port_2" default="50011"/>
+  <xacro:arg name="script_sender_port_2" default="50012"/>
+  <xacro:arg name="trajectory_port_2" default="50013"/>
+  <xacro:arg name="use_tool_communication" default="true"/>
   <xacro:arg name="tool_parity" default="0"/>
   <xacro:arg name="tool_baud_rate" default="115200"/>
@@ -56,10 +63,10 @@
     safety_k_position="$(arg safety_k_position)"
     >
-    <origin xyz="0.03 -0.0 0.65" rpy="0 0 ${pi}" />
+    <origin xyz="0.036 -0.0 1.0" rpy="0 0 ${-pi/4}" />
   </xacro:ur_robot>
   <!-- Mop tool attached to robot 1's tool0 -->
   <xacro:mop_tool prefix="" parent="$(arg tf_prefix)tool0" />
   <!-- ROBOT 2: second robot (no hardware interface, visualization only) -->
-   <xacro:ur_robot
+  <xacro:ur_robot
     name="ur_2"
     tf_prefix="ur_2_"
@@ -73,5 +80,5 @@
     safety_k_position="$(arg safety_k_position)"
     >
-    <origin xyz="0.0 -1.1 1.0" rpy="0 0 ${pi}" />
+    <origin xyz="0.0 -1.455 0.65" rpy="0 0 0.0" />
   </xacro:ur_robot>
   <xacro:robotiq_gripper
@@ -138,4 +145,32 @@
       trajectory_port="$(arg trajectory_port)"
     />
+    <xacro:ur_ros2_control
+      name="UR5ControlSystem_2"
+      tf_prefix="$(arg tf_prefix_2)"
+      kinematics_parameters_file="$(arg kinematics_params_2)"
+      transmission_hw_interface="$(arg transmission_hw_interface)"
+      use_mock_hardware="$(arg use_mock_hardware)"
+      mock_sensor_commands="$(arg mock_sensor_commands)"
+      headless_mode="$(arg headless_mode)"
+      initial_positions="${xacro.load_yaml(initial_positions_file)}"
+      use_tool_communication="$(arg use_tool_communication)"
+      tool_voltage="$(arg tool_voltage)"
+      tool_parity="$(arg tool_parity)"
+      tool_baud_rate="$(arg tool_baud_rate)"
+      tool_stop_bits="$(arg tool_stop_bits)"
+      tool_rx_idle_chars="$(arg tool_rx_idle_chars)"
+      tool_tx_idle_chars="$(arg tool_tx_idle_chars)"
+      tool_device_name="$(arg tool_device_name)"
+      tool_tcp_port="$(arg tool_tcp_port)"
+      robot_ip="$(arg robot_2_ip)"
+      script_filename="$(arg script_filename)"
+      output_recipe_filename="$(arg output_recipe_filename)"
+      input_recipe_filename="$(arg input_recipe_filename)"
+      reverse_ip="$(arg reverse_ip)"
+      script_command_port="$(arg script_command_port_2)"
+      reverse_port="$(arg reverse_port_2)"
+      script_sender_port="$(arg script_sender_port_2)"
+      trajectory_port="$(arg trajectory_port_2)"
+    />
   </xacro:unless>
   <xacro:if value="$(arg use_gazebo)">
@@ -204,5 +239,5 @@
         <state_interface name="velocity"/>
       </joint>
-<joint name="ur_2_robotiq_85_left_knuckle_joint">
+      <joint name="ur_2_robotiq_85_left_knuckle_joint">
         <command_interface name="position"/>
         <state_interface name="position"/>
@@ -240,5 +275,57 @@
     <parent link="world"/>
     <child link="table_link"/>
-    <origin rpy="0 0 ${pi}" xyz="0.0 -0.575 0.31"/>
+    <origin rpy="0 0 0" xyz="0.0 -0.675 0.31"/>
+  </joint>
+  <!-- Stand 1 -->
+  <link name="stand_1_link">
+    <visual>
+      <origin rpy="0 0 0" xyz="0.0 0.0 0.0"/>
+      <geometry>
+        <box size="0.495 0.495 1.0"/>
+      </geometry>
+      <material name="stand_material"><color rgba="0.6 0.4 0.2 1"/></material>
+    </visual>
+    <collision>
+      <origin rpy="0 0 0" xyz="0 0.0 0.0"/>
+      <geometry>
+        <box size="0.495 0.495 1.0"/>
+      </geometry>
+    </collision>
+    <inertial>
+      <mass value="10"/>
+      <origin rpy="0 0 0" xyz="0 0.0 0.0"/>
+      <inertia ixx="1" ixy="0" ixz="0" iyy="1" iyz="0" izz="1"/>
+    </inertial>
+  </link>
+  <joint name="world_to_stand_1" type="fixed">
+    <parent link="world"/>
+    <child link="stand_1_link"/>
+    <origin rpy="0 0 ${pi}" xyz="0.0 0.0 0.5"/>
+  </joint>
+  <!-- Stand 2 -->
+  <link name="stand_2_link">
+    <visual>
+      <origin rpy="0 0 0" xyz="0.0 0.0 0.0"/>
+      <geometry>
+        <box size="0.15 0.15 0.65"/>
+      </geometry>
+      <material name="stand_material"><color rgba="0.6 0.4 0.2 1"/></material>
+    </visual>
+    <collision>
+      <origin rpy="0 0 0" xyz="0 0.0 0.0"/>
+      <geometry>
+        <box size="0.15 0.15 0.65"/>
+      </geometry>
+    </collision>
+    <inertial>
+      <mass value="10"/>
+      <origin rpy="0 0 0" xyz="0 0.0 0.0"/>
+      <inertia ixx="1" ixy="0" ixz="0" iyy="1" iyz="0" izz="1"/>
+    </inertial>
+  </link>
+  <joint name="world_to_stand_2" type="fixed">
+    <parent link="world"/>
+    <child link="stand_2_link"/>
+    <origin rpy="0 0 ${pi}" xyz="0.0 -1.455 0.325"/>
   </joint>
 </robot>

File: src/ur_moveit_config/srdf/ur.srdf.xacro (robot description, xacro)
@@ -101,4 +101,8 @@
     <disable_collisions link1="ur_2_held_strip" link2="ur_2_robotiq_85_right_finger_tip_link" reason="Default"/>
     <disable_collisions link1="ur_2_base_link" link2="table_link" reason="Adjacent"/>
+    <disable_collisions link1="stand_1_link" link2="base_link" reason="Adjacent"/>
+    <disable_collisions link1="stand_1_link" link2="base_link_inertia" reason="Adjacent"/>
+    <disable_collisions link1="stand_2_link" link2="ur_2_base_link" reason="Adjacent"/>
+    <disable_collisions link1="stand_2_link" link2="ur_2_base_link_inertia" reason="Adjacent"/>
   <xacro:ur_srdf/>
 </robot>
