Commit message: fixed IK, Robot orientations, added wall, camera and everything else in the env. Planning works now

File: src/ur_description/urdf/inc/mop_tool.xacro (robot description, xacro)
@@ -5,9 +5,9 @@
       <parent link="${parent}" />
       <child link="${prefix}mop_handle" />
-      <origin xyz="-0.0 0.0 0.245" rpy="${pi/2} ${-pi} 0" />
+      <origin xyz="-0.0 0.0 0.245" rpy="0 0 0" />
     </joint>
     <link name="${prefix}mop_handle">
       <visual>
-        <origin xyz="0 0 0" rpy="${pi/2} ${-pi} 0" />
+        <origin xyz="0 0 0" rpy="0 ${-pi} 0" />
         <geometry>
           <cylinder radius="0.015" length="0.49" />
@@ -16,5 +16,5 @@
       </visual>
       <collision>
-        <origin xyz="0 0 0" rpy="${pi/2} ${-pi} 0" />
+        <origin xyz="0 0 0" rpy="0 ${-pi} 0" />
         <geometry>
           <cylinder radius="0.015" length="0.49" />
@@ -31,5 +31,5 @@
       <child link="${prefix}mop_dummy_r" />
       <axis xyz="1 0 0" />
-      <origin xyz="0 -0.245 -0.0" rpy="0 0 0" />
+      <origin xyz="0 0 0.245" rpy="0 0 0" />
       <dynamics damping="0.5" friction="0.01"/>
     </joint>
@@ -48,5 +48,5 @@
     <link name="${prefix}mop_head">
       <visual>
-        <origin xyz="-0.01 -0.01 -0.07" rpy="0 0 0" />
+        <origin xyz="-0.01 -0.07 0.01" rpy="${-pi/2} 0 0" />
         <geometry>
           <mesh filename="package://ur_description/meshes/mop_base.obj" scale="0.002 0.001 0.0015" />
@@ -55,5 +55,5 @@
       </visual>
       <collision>
-        <origin xyz="0 0 -0.0" rpy="${pi/2} ${-pi} 0"  />
+        <origin xyz="0 0 0.0" rpy="0 0 0"  />
         <geometry>
           <box size="0.25 0.13 0.02" />
@@ -68,5 +68,5 @@
       <parent link="${prefix}mop_handle"/>
       <child  link="${prefix}mop_tip"/>
-      <origin xyz="0  0.2 -0.00" rpy="${-pi/2}  0  ${pi}"/>
+      <origin xyz="0 -0.0 0.245" rpy="0 0 0"/>
     </joint>
     <link name="${prefix}mop_tip">

File: src/ur_description/urdf/ur_mop_standalone.urdf.xacro (robot description, xacro)
@@ -4,5 +4,5 @@
   <xacro:include filename="$(find ur_description)/urdf/inc/mop_tool.xacro"/>
   <!-- ADDED: official ros2_control macro that has ALL required params -->
-  <xacro:include filename="$(find robotiq_description)/urdf/robotiq_2f_85_macro.urdf.xacro"/>
+  <!-- <xacro:include filename="$(find robotiq_description)/urdf/robotiq_2f_85_macro.urdf.xacro"/> -->
   <xacro:include filename="$(find ur_robot_driver)/urdf/ur.ros2_control.xacro"/>
   <xacro:arg name="ur_type" default="ur5"/>
@@ -80,7 +80,7 @@
     safety_k_position="$(arg safety_k_position)"
     >
-    <origin xyz="0.0 -1.455 0.65" rpy="0 0 0.0" />
+    <origin xyz="0.0 -1.44 0.65" rpy="0 0 0.0" />
   </xacro:ur_robot>
-  <xacro:robotiq_gripper
+  <!-- <xacro:robotiq_gripper
     name="ur_2_robotiq_85"
     prefix="ur_2_"
@@ -88,16 +88,16 @@
     include_ros2_control="false"    >
     <origin xyz="0 0 0" rpy="0 0 0" />
-  </xacro:robotiq_gripper>
-  <link name="ur_2_held_strip">
-    <visual>
-      <geometry>
-        <box size="0.15 0.7 0.012"/>
-      </geometry>
-      <material name="strip_color">
-        <color rgba="0.1 0.1 0.8 1.0"/> </material>
-    </visual>
-    <collision>
-      <geometry>
-        <box size="0.15 0.7 0.012"/>
+  </xacro:robotiq_gripper> -->
+   <link name="ur_2_gripper">
+    <visual>
+      <geometry>
+        <box size="0.13 0.05 0.07"/>
+      </geometry>
+      <material name="gripper_color">
+        <color rgba="0.7 0.71 0.8 1.0"/> </material>
+    </visual>
+    <collision>
+      <geometry>
+        <box size="0.13 0.05 0.07"/>
       </geometry>
     </collision>
@@ -108,6 +108,30 @@
     </inertial>
   </link>
+    <joint name="ur_2_gripper_joint" type="fixed">
+    <parent link="ur_2_tool0"/>
+    <child link="ur_2_gripper"/>
+    <origin xyz="0 0 0.04" rpy="0 ${pi/2} 0"/>
+  </joint>
+  <link name="ur_2_held_strip">
+    <visual>
+      <geometry>
+        <box size="0.15 0.7 0.012"/>
+      </geometry>
+      <material name="strip_color">
+        <color rgba="0.1 0.1 0.8 1.0"/> </material>
+    </visual>
+    <collision>
+      <geometry>
+        <box size="0.15 0.7 0.012"/>
+      </geometry>
+    </collision>
+    <inertial>
+      <mass value="0.2"/>
+      <origin xyz="0 0 0" rpy="0 0 0"/>
+      <inertia ixx="0.001" ixy="0" ixz="0" iyy="0.001" iyz="0" izz="0.001"/>
+    </inertial>
+  </link>
   <joint name="ur_2_to_strip" type="fixed">
-    <parent link="ur_2_robotiq_85_base_link"/>
+    <parent link="ur_2_tool0"/>
     <child link="ur_2_held_strip"/>
     <origin xyz="0 0 0.18" rpy="0 ${pi/2} 0"/>
@@ -239,9 +263,4 @@
         <state_interface name="velocity"/>
       </joint>
-      <joint name="ur_2_robotiq_85_left_knuckle_joint">
-        <command_interface name="position"/>
-        <state_interface name="position"/>
-        <state_interface name="velocity"/>
-      </joint>
     </ros2_control>
     <gazebo>
@@ -329,3 +348,105 @@
     <origin rpy="0 0 ${pi}" xyz="0.0 -1.455 0.325"/>
   </joint>
+  <!-- Wall -->
+  <link name="wall_link">
+    <visual>
+      <origin rpy="0 0 0" xyz="0.0 0.0 0.0"/>
+      <geometry>
+        <box size="3.5 0.2 3.5"/>
+      </geometry>
+      <material name="wall_material"><color rgba="0.8 0.8 0.8 1"/></material>
+    </visual>
+    <collision>
+      <origin rpy="0 0 0" xyz="0.0 0.0 0.0"/>
+      <geometry>
+        <box size="3.5 0.2 3.5"/>
+      </geometry>
+    </collision>
+    <inertial>
+      <mass value="50"/>
+      <origin rpy="0 0 0" xyz="0.0 -1.455 1.25"/>
+      <inertia ixx="10" ixy="0" ixz="0" iyy="10" iyz="0" izz="10"/>
+    </inertial>
+  </link>
+  <joint name="world_to_wall" type="fixed">
+    <parent link="world"/>
+    <child link="wall_link"/>
+    <origin rpy="0 0 ${pi}" xyz="0.0 0.545 1.25"/>
+  </joint>
+  <!-- Camera setup -->
+  <link name="camera_link">
+    <visual>
+      <origin rpy="0 0 0" xyz="0.0 0.0 0.0"/>
+      <geometry>
+        <box size="0.1 0.1 0.1"/>
+      </geometry>
+      <material name="camera_material"><color rgba="0.2 0.2 0.2 1"/></material>
+    </visual>
+    <collision>
+      <origin rpy="0 0 0" xyz="0.0 0.0 0.0"/>
+      <geometry>
+        <box size="0.1 0.1 0.1"/>
+      </geometry>
+    </collision>
+    <inertial>
+      <mass value="1"/>
+      <origin rpy="0 0 0" xyz="0.0 0.0 0.5"/>
+      <inertia ixx="1" ixy="1" ixz="1" iyy="1" iyz="1" izz="1"/>
+    </inertial>
+  </link>
+  <link name="camera_optical_link_1">
+    <visual>
+      <origin rpy="0 0 0" xyz="0.0 0.0 0.0"/>
+      <geometry>
+        <cylinder length="0.60" radius="0.025"/>
+      </geometry>
+      <material name="camera_material"><color rgba="0.2 0.2 0.2 1"/></material>
+    </visual>
+    <collision>
+      <origin rpy="0 0 0" xyz="0.0 0.0 0.0"/>
+      <geometry>
+        <cylinder length="0.60" radius="0.025"/>
+      </geometry>
+    </collision>
+    <inertial>
+      <mass value="1"/>
+      <origin rpy="0 0 0" xyz="0.0 0.05 0.5"/>
+      <inertia ixx="1" ixy="1" ixz="1" iyy="1" iyz="1" izz="1"/>
+    </inertial>
+  </link>
+  <link name="camera_optical_link_2">
+    <visual>
+      <origin rpy="0 0 0" xyz="0.0 0.0 0.0"/>
+      <geometry>
+        <cylinder length="1.23" radius="0.025"/>
+      </geometry>
+      <material name="camera_material"><color rgba="0.2 0.2 0.2 1"/></material>
+    </visual>
+    <collision>
+      <origin rpy="0 0 0" xyz="0.0 0.0 0.0"/>
+      <geometry>
+        <cylinder length="1.23" radius="0.025"/>
+      </geometry>
+    </collision>
+    <inertial>
+      <mass value="1"/>
+      <origin rpy="0 0 0" xyz="-0.05 0.05 0.5"/>
+      <inertia ixx="1" ixy="1" ixz="1" iyy="1" iyz="1" izz="1"/>
+    </inertial>
+  </link>
+  <joint name="camera_to_optical_1" type="fixed">
+    <parent link="camera_link"/>
+    <child link="camera_optical_link_1"/>
+    <origin rpy="0 ${pi/2} 0" xyz="-0.3 0.0 0.0"/>
+  </joint>
+  <joint name="camera_to_optical_2" type="fixed">
+    <parent link="camera_optical_link_1"/>
+    <child link="camera_optical_link_2"/>
+    <origin rpy="${pi/2} 0 0" xyz="0.0 0.615 -0.3"/>
+  </joint>
+  <joint name="world_to_camera" type="fixed">
+    <parent link="world"/>
+    <child link="camera_link"/>
+    <origin rpy="0 ${pi/2} 0" xyz="0.0 -0.86 1.57"/>
+  </joint>
 </robot>

File: src/ur_moveit_config/srdf/ur.srdf.xacro (robot description, xacro)
@@ -9,5 +9,5 @@
     <disable_collisions link1="mop_head" link2="table_link" reason="Never" />
     <disable_collisions link1="mop_tip" link2="table_link" reason="Never" />
-    <disable_collisions link1="ur_2_robotiq_85_base_link" link2="ur_2_wrist_3_link" reason="Adjacent"/>
+    <!-- <disable_collisions link1="ur_2_robotiq_85_base_link" link2="ur_2_wrist_3_link" reason="Adjacent"/>
     <disable_collisions link1="ur_2_robotiq_85_left_knuckle_link" link2="ur_2_wrist_3_link" reason="Never"/>
     <disable_collisions  link1="ur_2_robotiq_85_right_knuckle_link" link2="ur_2_wrist_3_link" reason="Never"/>
@@ -99,10 +99,21 @@
     <disable_collisions link1="ur_2_held_strip" link2="ur_2_robotiq_85_right_finger_link" reason="Never"/>
     <disable_collisions link1="ur_2_held_strip" link2="ur_2_robotiq_85_left_finger_tip_link" reason="Default"/>
-    <disable_collisions link1="ur_2_held_strip" link2="ur_2_robotiq_85_right_finger_tip_link" reason="Default"/>
+    <disable_collisions link1="ur_2_held_strip" link2="ur_2_robotiq_85_right_finger_tip_link" reason="Default"/> -->
     <disable_collisions link1="ur_2_base_link" link2="table_link" reason="Adjacent"/>
+     <disable_collisions link1="ur_2_gripper" link2="ur_2_wrist_3_link" reason="Adjacent" />
+      <disable_collisions link1="ur_2_gripper" link2="ur_2_tool0" reason="Adjacent" />
+            <disable_collisions link1="ur_2_gripper" link2="ur_2_tool0" reason="Adjacent" />
+      <disable_collisions link1="ur_2_gripper" link2="ur_2_held_strip" reason="Adjacent" />
+            <disable_collisions link1="ur_2_gripper" link2="table_link" reason="Adjacent" />
+      <!-- <disable_collisions link1="ur_2_held_strip" link2="table_link" reason="Adjacent"/> -->
     <disable_collisions link1="stand_1_link" link2="base_link" reason="Adjacent"/>
     <disable_collisions link1="stand_1_link" link2="base_link_inertia" reason="Adjacent"/>
+      <!-- <disable_collisions link1="stand_1_link" link2="upper_arm_link" reason="Never"/> -->
     <disable_collisions link1="stand_2_link" link2="ur_2_base_link" reason="Adjacent"/>
     <disable_collisions link1="stand_2_link" link2="ur_2_base_link_inertia" reason="Adjacent"/>
+    <!-- disable camera self-collisions -->
+    <disable_collisions link1="camera_optical_link_1" link2="camera_optical_link_2" reason="Adjacent"/>
+    <disable_collisions link1="camera_link" link2="camera_optical_link_1" reason="Adjacent"/>
+    <!-- <disable_collisions link1="ur_2_camera_link" link2="ur_2_shoulder_link" reason="Adjacent"/> -->
   <xacro:ur_srdf/>
 </robot>
