Commit message: updated orientation of the robot

File: src/ur_description/urdf/ur_mop_standalone.urdf.xacro (robot description, xacro)
@@ -301,5 +301,5 @@
       <origin rpy="0 0 0" xyz="0.0 0.0 0.0"/>
       <geometry>
-        <box size="0.495 0.495 1.0"/>
+        <box size="0.5 0.5 1.0"/>
       </geometry>
       <material name="stand_material"><color rgba="0.6 0.4 0.2 1"/></material>
@@ -308,5 +308,5 @@
       <origin rpy="0 0 0" xyz="0 0.0 0.0"/>
       <geometry>
-        <box size="0.495 0.495 1.0"/>
+        <box size="0.5 0.5 1.0"/>
       </geometry>
     </collision>
